Commit message: [kinova_description] j2s6s200: Simplified meshes

File: kinova_description/urdf/j2s6s200.xacro (robot description, xacro)
@@ -104,17 +104,17 @@
     <xacro:macro name="j2s6s200" params="base_parent prefix:=j2s6s200">
         <xacro:gazebo_config robot_namespace="${prefix}"/>
-        <xacro:kinova_armlink link_name="${prefix}_link_base" link_mesh="${link_base_mesh}" mesh_no="${link_base_mesh_no}"/>
+        <xacro:kinova_armlink_base link_name="${prefix}_link_base" link_mesh="${link_base_mesh}" mesh_no="${link_base_mesh_no}"/>
         <xacro:kinova_armjoint joint_name="${prefix}_joint_base" type="${joint_base_type}" parent="${base_parent}" child="${prefix}_link_base" joint_axis_xyz="${joint_base_axis_xyz}" joint_origin_xyz="${joint_base_origin_xyz}" joint_origin_rpy="${joint_base_origin_rpy}" joint_lower_limit="0" joint_upper_limit="0" joint_velocity_limit="0" joint_torque_limit="0" fixed="true"/>
-        <xacro:kinova_armlink link_name="${prefix}_link_1" link_mesh="${link_1_mesh}" use_ring_mesh="true" mesh_no="${link_1_mesh_no}"/>
+        <xacro:kinova_armlink_shoulder link_name="${prefix}_link_1" link_mesh="${link_1_mesh}" use_ring_mesh="true" mesh_no="${link_1_mesh_no}"/>
         <xacro:kinova_armjoint joint_name="${prefix}_joint_1" type="${joint_1_type}" parent="${prefix}_link_base" child="${prefix}_link_1" joint_axis_xyz="${joint_1_axis_xyz}" joint_origin_xyz="${joint_1_origin_xyz}" joint_origin_rpy="${joint_1_origin_rpy}" joint_lower_limit="${joint_1_lower_limit}" joint_upper_limit="${joint_1_upper_limit}" joint_velocity_limit="${joint_1_velocity_limit}" joint_torque_limit="${joint_1_torque_limit}"/>
-        <xacro:kinova_armlink link_name="${prefix}_link_2" link_mesh="${link_2_mesh}" use_ring_mesh="true" mesh_no="${link_2_mesh_no}"/>
+        <xacro:kinova_armlink_arm link_name="${prefix}_link_2" link_mesh="${link_2_mesh}" use_ring_mesh="true" mesh_no="${link_2_mesh_no}"/>
         <xacro:kinova_armjoint joint_name="${prefix}_joint_2" type="${joint_2_type}" parent="${prefix}_link_1" child="${prefix}_link_2" joint_axis_xyz="${joint_2_axis_xyz}" joint_origin_xyz="${joint_2_origin_xyz}" joint_origin_rpy="${joint_2_origin_rpy}" joint_lower_limit="${joint_2_lower_limit}" joint_upper_limit="${joint_2_upper_limit}" joint_velocity_limit="${joint_2_velocity_limit}" joint_torque_limit="${joint_2_torque_limit}"/>
-        <xacro:kinova_armlink link_name="${prefix}_link_3" link_mesh="${link_3_mesh}" use_ring_mesh="true" mesh_no="${link_3_mesh_no}"/>
+        <xacro:kinova_armlink_forearm link_name="${prefix}_link_3" link_mesh="${link_3_mesh}" use_ring_mesh="true" mesh_no="${link_3_mesh_no}"/>
         <xacro:kinova_armjoint joint_name="${prefix}_joint_3" type="${joint_3_type}" parent="${prefix}_link_2" child="${prefix}_link_3" joint_axis_xyz="${joint_3_axis_xyz}" joint_origin_xyz="${joint_3_origin_xyz}" joint_origin_rpy="${joint_3_origin_rpy}" joint_lower_limit="${joint_3_lower_limit}" joint_upper_limit="${joint_3_upper_limit}" joint_velocity_limit="${joint_3_velocity_limit}" joint_torque_limit="${joint_3_torque_limit}"/>
-        <xacro:kinova_armlink link_name="${prefix}_link_4" link_mesh="${link_4_mesh}" use_ring_mesh="true" ring_mesh="ring_small" mesh_no="${link_4_mesh_no}"/>
+        <xacro:kinova_armlink_wrist_spherical_1 link_name="${prefix}_link_4" link_mesh="${link_4_mesh}" use_ring_mesh="true" ring_mesh="ring_small" mesh_no="${link_4_mesh_no}"/>
         <xacro:kinova_armjoint joint_name="${prefix}_joint_4" type="${joint_4_type}" parent="${prefix}_link_3" child="${prefix}_link_4" joint_axis_xyz="${joint_4_axis_xyz}" joint_origin_xyz="${joint_4_origin_xyz}" joint_origin_rpy="${joint_4_origin_rpy}" joint_lower_limit="${joint_4_lower_limit}" joint_upper_limit="${joint_4_upper_limit}" joint_velocity_limit="${joint_4_velocity_limit}" joint_torque_limit="${joint_4_torque_limit}"/>
-        <xacro:kinova_armlink link_name="${prefix}_link_5" link_mesh="${link_5_mesh}" use_ring_mesh="true" ring_mesh="ring_small" mesh_no="${link_5_mesh_no}"/>
+        <xacro:kinova_armlink_wrist_spherical_2 link_name="${prefix}_link_5" link_mesh="${link_5_mesh}" use_ring_mesh="true" ring_mesh="ring_small" mesh_no="${link_5_mesh_no}"/>
         <xacro:kinova_armjoint joint_name="${prefix}_joint_5" type="${joint_5_type}" parent="${prefix}_link_4" child="${prefix}_link_5" joint_axis_xyz="${joint_5_axis_xyz}" joint_origin_xyz="${joint_5_origin_xyz}" joint_origin_rpy="${joint_5_origin_rpy}" joint_lower_limit="${joint_5_lower_limit}" joint_upper_limit="${joint_5_upper_limit}" joint_velocity_limit="${joint_5_velocity_limit}" joint_torque_limit="${joint_5_torque_limit}"/>
-        <xacro:kinova_armlink link_name="${prefix}_link_6" link_mesh="${link_6_mesh}" use_ring_mesh="true" ring_mesh="ring_small" mesh_no="${link_6_mesh_no}"/>
+        <xacro:kinova_armlink_hand_2finger link_name="${prefix}_link_6" link_mesh="${link_6_mesh}" use_ring_mesh="true" ring_mesh="ring_small" mesh_no="${link_6_mesh_no}"/>
         <xacro:kinova_armjoint joint_name="${prefix}_joint_6" type="${joint_6_type}" parent="${prefix}_link_5" child="${prefix}_link_6" joint_axis_xyz="${joint_6_axis_xyz}" joint_origin_xyz="${joint_6_origin_xyz}" joint_origin_rpy="${joint_6_origin_rpy}" joint_lower_limit="${joint_6_lower_limit}" joint_upper_limit="${joint_6_upper_limit}" joint_velocity_limit="${joint_6_velocity_limit}" joint_torque_limit="${joint_6_torque_limit}"/>
         <xacro:kinova_virtual_link link_name="${prefix}_end_effector"/>

File: kinova_description/urdf/kinova_common.xacro (robot description, xacro)
@@ -13,6 +13,6 @@
     xmlns:physics="http://playerstage.sourceforge.net/gazebo/xmlschema/#physics"
 	xmlns:xacro="http://www.ros.org/wiki/xacro">
-<xacro:include filename="$(find kinova_description)/urdf/kinova_inertial.xacro" />
-    <xacro:property name="J_PI" value="3.1415926535897931" />
+  <xacro:include filename="$(find kinova_description)/urdf/kinova_inertial.xacro" />
+  <xacro:property name="J_PI" value="3.1415926535897931" />
     <xacro:macro name="kinova_armlink" params="link_name link_mesh ring_mesh:=ring_big use_ring_mesh:=false mesh_no">
         <link name="${link_name}">
@@ -35,13 +35,206 @@
              </visual>
 	    </xacro:if>
-            <collision>
+            <!-- <collision>
                 <geometry>
+                    <mesh filename="package://kinova_description/meshes/collision/${link_mesh}.stl"/>
                     <mesh
-                        filename="package://kinova_description/meshes/${link_mesh}.dae"/>
+                      filename="package://kinova_description/meshes/${link_mesh}.dae"/>
                 </geometry>
-            </collision>
+            </collision> -->
 						<xacro:kinova_inertial mesh_no="${mesh_no}"/>
       </link>
     </xacro:macro>
+  <xacro:macro name="kinova_armlink_base" params="link_name link_mesh ring_mesh:=ring_big use_ring_mesh:=false mesh_no">
+    <link name="${link_name}">
+      <visual>
+        <geometry>
+          <mesh filename="package://kinova_description/meshes/${link_mesh}.dae"/>
+        </geometry>
+        <material name="carbon_fiber">
+          <color rgba="0.792156862745098 0.819607843137255 0.933333333333333 1" />
+        </material>
+      </visual>
+      <!-- Adding ring to the model -->
+      <xacro:if value="${use_ring_mesh}">
+        <visual>
+          <geometry>
+            <mesh filename="package://kinova_description/meshes/${ring_mesh}.dae"/>
+          </geometry>
+        </visual>
+      </xacro:if>
+      <collision>
+        <origin xyz="0 0 0.078375" rpy="0 0 0"/>
+        <geometry>
+          <cylinder radius="0.04125" length="0.156750"/>
+        </geometry>
+      </collision>
+      <xacro:kinova_inertial mesh_no="${mesh_no}"/>
+    </link>
+  </xacro:macro>
+  <xacro:macro name="kinova_armlink_shoulder" params="link_name link_mesh ring_mesh:=ring_big use_ring_mesh:=false mesh_no">
+    <link name="${link_name}">
+      <visual>
+        <geometry>
+          <mesh filename="package://kinova_description/meshes/${link_mesh}.dae"/>
+        </geometry>
+        <material name="carbon_fiber">
+          <color rgba="0.792156862745098 0.819607843137255 0.933333333333333 1" />
+        </material>
+      </visual>
+      <!-- Adding ring to the model -->
+      <xacro:if value="${use_ring_mesh}">
+        <visual>
+          <geometry>
+            <mesh filename="package://kinova_description/meshes/${ring_mesh}.dae"/>
+          </geometry>
+        </visual>
+      </xacro:if>
+      <collision>
+        <origin xyz="0 0 -0.08" rpy="0 0 0"/>
+        <geometry>
+          <cylinder radius="0.05" length="0.16"/>
+        </geometry>
+      </collision>
+      <xacro:kinova_inertial mesh_no="${mesh_no}"/>
+    </link>
+  </xacro:macro>
+  <xacro:macro name="kinova_armlink_arm" params="link_name link_mesh ring_mesh:=ring_big use_ring_mesh:=false mesh_no">
+    <link name="${link_name}">
+      <visual>
+        <geometry>
+          <mesh filename="package://kinova_description/meshes/${link_mesh}.dae"/>
+        </geometry>
+        <material name="carbon_fiber">
+          <color rgba="0.792156862745098 0.819607843137255 0.933333333333333 1" />
+        </material>
+      </visual>
+      <!-- Adding ring to the model -->
+      <xacro:if value="${use_ring_mesh}">
+        <visual>
+          <geometry>
+            <mesh filename="package://kinova_description/meshes/${ring_mesh}.dae"/>
+          </geometry>
+        </visual>
+      </xacro:if>
+      <collision>
+        <origin xyz="0 ${-0.25+0.04125} 0" rpy="${J_PI/2} 0 0"/>
+        <geometry>
+          <cylinder radius="0.05" length="0.50"/>
+        </geometry>
+      </collision>
+      <xacro:kinova_inertial mesh_no="${mesh_no}"/>
+    </link>
+  </xacro:macro>
+  <xacro:macro name="kinova_armlink_forearm" params="link_name link_mesh ring_mesh:=ring_big use_ring_mesh:=false mesh_no">
+    <link name="${link_name}">
+      <visual>
+        <geometry>
+          <mesh filename="package://kinova_description/meshes/${link_mesh}.dae"/>
+        </geometry>
+        <material name="carbon_fiber">
+          <color rgba="0.792156862745098 0.819607843137255 0.933333333333333 1" />
+        </material>
+      </visual>
+      <!-- Adding ring to the model -->
+      <xacro:if value="${use_ring_mesh}">
+        <visual>
+          <geometry>
+            <mesh filename="package://kinova_description/meshes/${ring_mesh}.dae"/>
+          </geometry>
+        </visual>
+      </xacro:if>
+      <collision>
+        <origin xyz="0 ${0.125-0.04125} 0" rpy="${J_PI/2} 0 0"/>
+        <geometry>
+          <cylinder radius="0.05" length="0.25"/>
+        </geometry>
+      </collision>
+      <xacro:kinova_inertial mesh_no="${mesh_no}"/>
+    </link>
+  </xacro:macro>
+  <!-- wrist_spherical_1 -->
+  <xacro:macro name="kinova_armlink_wrist_spherical_1" params="link_name link_mesh ring_mesh:=ring_big use_ring_mesh:=false mesh_no">
+    <link name="${link_name}">
+      <visual>
+        <geometry>
+          <mesh filename="package://kinova_description/meshes/${link_mesh}.dae"/>
+        </geometry>
+        <material name="carbon_fiber">
+          <color rgba="0.792156862745098 0.819607843137255 0.933333333333333 1" />
+        </material>
+      </visual>
+      <!-- Adding ring to the model -->
+      <xacro:if value="${use_ring_mesh}">
+        <visual>
+          <geometry>
+            <mesh filename="package://kinova_description/meshes/${ring_mesh}.dae"/>
+          </geometry>
+        </visual>
+      </xacro:if>
+      <collision>
+        <origin xyz="0 0 -0.07" rpy="0 0 0"/>
+        <geometry>
+          <cylinder radius="0.05" length="0.14"/>
+        </geometry>
+      </collision>
+      <xacro:kinova_inertial mesh_no="${mesh_no}"/>
+    </link>
+  </xacro:macro>
+  <!-- wrist_spherical_2 -->
+  <xacro:macro name="kinova_armlink_wrist_spherical_2" params="link_name link_mesh ring_mesh:=ring_big use_ring_mesh:=false mesh_no">
+    <link name="${link_name}">
+      <visual>
+        <geometry>
+          <mesh filename="package://kinova_description/meshes/${link_mesh}.dae"/>
+        </geometry>
+        <material name="carbon_fiber">
+          <color rgba="0.792156862745098 0.819607843137255 0.933333333333333 1" />
+        </material>
+      </visual>
+      <!-- Adding ring to the model -->
+      <xacro:if value="${use_ring_mesh}">
+        <visual>
+          <geometry>
+            <mesh filename="package://kinova_description/meshes/${ring_mesh}.dae"/>
+          </geometry>
+        </visual>
+      </xacro:if>
+      <collision>
+        <origin xyz="0 0.045 0" rpy="${J_PI/2} 0 0"/>
+        <geometry>
+          <cylinder radius="0.05" length="0.14"/>
+        </geometry>
+      </collision>
+      <xacro:kinova_inertial mesh_no="${mesh_no}"/>
+    </link>
+  </xacro:macro>
+  <!-- hand_2finger -->
+  <xacro:macro name="kinova_armlink_hand_2finger" params="link_name link_mesh ring_mesh:=ring_big use_ring_mesh:=false mesh_no">
+    <link name="${link_name}">
+      <visual>
+        <geometry>
+          <mesh filename="package://kinova_description/meshes/${link_mesh}.dae"/>
+        </geometry>
+        <material name="carbon_fiber">
+          <color rgba="0.792156862745098 0.819607843137255 0.933333333333333 1" />
+        </material>
+      </visual>
+      <!-- Adding ring to the model -->
+      <xacro:if value="${use_ring_mesh}">
+        <visual>
+          <geometry>
+            <mesh filename="package://kinova_description/meshes/${ring_mesh}.dae"/>
+          </geometry>
+        </visual>
+      </xacro:if>
+      <collision>
+        <origin xyz="0 0 -${.125/2}" rpy="0 0 0"/>
+        <geometry>
+          <box size="0.065 0.11 0.125"/>
+        </geometry>
+      </collision>
+      <xacro:kinova_inertial mesh_no="${mesh_no}"/>
+    </link>
+  </xacro:macro>
   <xacro:macro name="kinova_armjoint" params="joint_name type parent child joint_axis_xyz joint_origin_xyz joint_origin_rpy joint_lower_limit joint_upper_limit joint_velocity_limit joint_torque_limit fixed:=false">
     <joint name="${joint_name}" type="${type}">
